Commit message: add geometry macros with meshes

File: cob_description/urdf/common.xacro (robot description, xacro)
@@ -2,4 +2,9 @@
 <robot xmlns:xacro="http://www.ros.org/wiki/xacro">
   <property name="M_PI" value="3.1415926535897931" />
+  <xacro:macro name="box_geometry" params="x y z">
+    <geometry>
+      <mesh filename="package://cob_description/meshes/box_1.0.stl" scale="${x} ${y} ${z}"/>
+    </geometry>
+  </xacro:macro>
   <!-- see https://secure.wikimedia.org/wikipedia/en/wiki/List_of_moment_of_inertia_tensors -->
   <xacro:macro name="sphere_inertial" params="radius mass *origin">
